File: pcb/paaliaq-pcb.kicad_pcb (KiCad board)
At the start: 2 copper layers, 3 parts, among them J1 SODIMM-200, J2 HDMI_A, U1 W65C816SxP

Commit message: wip pcb
Parts:
- added C1: 1uF, Capacitor_SMD:C_0805_2012Metric_Pad1.18x1.45mm_HandSolder, F.Cu at (71.1, 111.9)
- added C2: 4.7uF, Capacitor_SMD:C_0805_2012Metric_Pad1.18x1.45mm_HandSolder, F.Cu at (57.6, 114.3)
- added C3: 1000pF, Capacitor_SMD:C_0805_2012Metric_Pad1.18x1.45mm_HandSolder, F.Cu at (71.1, 116.6)
- added R1: 1k, Resistor_SMD:R_0805_2012Metric_Pad1.20x1.40mm_HandSolder, F.Cu at (60.2, 114.3)
- added U3: MCP1727-3302xSN, Package_SO:SOIC-8_3.9x4.9mm_P1.27mm, F.Cu at (65.8, 114.9)
Routing:
- net +5V: track 0.00 -> 7.15 mm
- net +3.3V: track 0.00 -> 4.09 mm
- net Net-(U3-~{SHDN}): track 0.00 -> 3.25 mm
- net Net-(U3-Cdelay): track 0.00 -> 2.81 mm
Other:
- board outline added: 100 x 100 mm

Commit message: wip dvi phy
Parts:
- added R2: 270, Resistor_SMD:R_0603_1608Metric_Pad0.98x0.95mm_HandSolder, F.Cu at (136.7, 62.0)
- added R3: 270, Resistor_SMD:R_0603_1608Metric_Pad0.98x0.95mm_HandSolder, F.Cu at (136.7, 63.5)
- added R4: 270, Resistor_SMD:R_0603_1608Metric_Pad0.98x0.95mm_HandSolder, F.Cu at (130.7, 64.0)
- added R5: 270, Resistor_SMD:R_0603_1608Metric_Pad0.98x0.95mm_HandSolder, F.Cu at (130.7, 65.5)
- added R6: 270, Resistor_SMD:R_0603_1608Metric_Pad0.98x0.95mm_HandSolder, F.Cu at (136.7, 66.0)
- added R7: 270, Resistor_SMD:R_0603_1608Metric_Pad0.98x0.95mm_HandSolder, F.Cu at (136.7, 67.5)
- added R8: 270, Resistor_SMD:R_0603_1608Metric_Pad0.98x0.95mm_HandSolder, F.Cu at (130.7, 68.5)
- added R9: 270, Resistor_SMD:R_0603_1608Metric_Pad0.98x0.95mm_HandSolder, F.Cu at (130.7, 70.0)
- moved J2 29.5 mm to (146.2, 67.5)
Connections:
- J2 pad 1: /HDMI_D2+ -> /xHDMI_D2+
- J2 pad 10: /HDMI_CK+ -> /xHDMI_CK+
- J2 pad 12: /HDMI_CK- -> /xHDMI_CK-
- J2 pad 3: /HDMI_D2- -> /xHDMI_D2-
- J2 pad 4: /HDMI_D1+ -> /xHDMI_D1+
- J2 pad 6: /HDMI_D1- -> /xHDMI_D1-
- J2 pad 7: /HDMI_D0+ -> /xHDMI_D0+
- J2 pad 9: /HDMI_D0- -> /xHDMI_D0-
Routing:
- net /HDMI_CK-: track 45.6 -> 5.43 mm
- net /HDMI_CK+: track 45.5 -> 5.80 mm
- net /HDMI_D1-: track 43.4 -> 7.82 mm
- net /HDMI_D1+: track 43.5 -> 8.19 mm
- net /HDMI_D0-: track 46.2 -> 12.6 mm
- net /HDMI_D0+: track 46.2 -> 13.0 mm
- net /HDMI_D2-: track 46.5 -> 15.0 mm
- net /HDMI_D2+: track 46.5 -> 15.4 mm
- net /xHDMI_CK-: track 0.00 -> 10.5 mm
- net /xHDMI_CK+: track 0.00 -> 10.5 mm
- net /xHDMI_D1-: track 0.00 -> 9.92 mm
- net /xHDMI_D1+: track 0.00 -> 9.92 mm
- net /xHDMI_D0+: track 0.00 -> 4.13 mm
- net /xHDMI_D2-: track 0.00 -> 4.13 mm
- net /xHDMI_D2+: track 0.00 -> 4.13 mm
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
Commit message: wip use resistor arrays and swap pairs and +/-
Parts:
- removed R2, R3, R4, R5, R6, R7, R8, R9: 270, Resistor_SMD:R_0603_1608Metric_Pad0.98x0.95mm_HandSolder
- added RN1: 270, Resistor_SMD:R_Array_Convex_4x1206, F.Cu at (108.5, 115.0)
- added RN2: 270, Resistor_SMD:R_Array_Convex_4x1206, F.Cu at (102.5, 115.0)
- moved J2 73.1 mm to (104.5, 127.5), turned to 0 degrees
- moved U1 53.9 mm to (79.5, 69.5)
- moved C3 9.11 mm to (71.1, 125.7)
- moved R1 9.11 mm to (60.2, 123.4)
- moved U3 9.11 mm to (65.8, 124.0)
- moved C1 9.10 mm to (71.1, 121.0)
- moved C2 9.10 mm to (57.6, 123.4)
- moved J1 6.05 mm to (99.9, 103.6)
Connections:
- J1 pad 103: /HDMI_D2+ -> /HDMI_CK-
- J1 pad 109: /HDMI_D2- -> /HDMI_CK+
- J1 pad 111: /HDMI_D1+ -> /HDMI_D0-
- J1 pad 113: /HDMI_D1- -> /HDMI_D0+
- J1 pad 115: /HDMI_D0+ -> /HDMI_D1-
- J1 pad 117: /HDMI_D0- -> /HDMI_D1+
- J1 pad 119: /HDMI_CK+ -> /HDMI_D2-
- J1 pad 121: /HDMI_CK- -> /HDMI_D2+
Routing:
- net GND: track 21.2 -> 0.00 mm
- net /HDMI_D2+: track 15.4 -> 0.00 mm
- net /HDMI_D2-: track 15.0 -> 0.00 mm
- net /HDMI_D0+: track 13.0 -> 0.00 mm
- net /HDMI_D0-: track 12.6 -> 0.00 mm
- net /xHDMI_CK-: track 10.5 -> 0.80 mm
- net /xHDMI_CK+: track 10.5 -> 0.80 mm
- net /xHDMI_D1-: track 9.92 -> 1.43 mm
- net /xHDMI_D1+: track 9.92 -> 1.43 mm
- net /HDMI_D1+: track 8.19 -> 0.00 mm
- net /HDMI_D1-: track 7.82 -> 0.00 mm
- net +5V: track 7.15 -> 0.44 mm
- net /HDMI_CK+: track 5.80 -> 0.00 mm
- net /HDMI_CK-: track 5.43 -> 0.00 mm
- net Net-(U3-~{SHDN}): track 3.25 -> 0.33 mm
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